File: kicad/mqtt_particle_sensor.kicad_pcb (KiCad board)
At the start: 2 copper layers, 91.4 x 66 mm, 26 parts, among them J2 Barrel_Jack, Q1 2N7000, Q2 2N7000, U1 CD4060BM96, U3 HPM_Particle_Sensor

Commit message: revC
Parts:
- added R8: 4k7, Resistor_SMD:R_1206_3216Metric_Pad1.30x1.75mm_HandSolder, F.Cu at (49.2, 71.1)
- added R9: 4k7, Resistor_SMD:R_1206_3216Metric_Pad1.30x1.75mm_HandSolder, F.Cu at (49.2, 76.2)
- added REF**: OSHW-Logo2_14.6x12mm_SilkScreen, Symbol:OSHW-Logo2_14.6x12mm_SilkScreen, B.Cu at (99.1, 92.7)
- added U2: ATtiny85-20P, Package_DIP:DIP-8_W7.62mm, F.Cu at (47.0, 82.6)
Connections:
- A1 pad 14: HPM_RESET -> unconnected-(A1-15-Pad14)
- A1 pad 17: unconnected-(A1-4-Pad17) -> SDA
- A1 pad 18: unconnected-(A1-5-Pad18) -> SCL
- A1 pad 19: UART_MISO -> unconnected-(A1-RX-Pad19)
- A1 pad 20: UART_MOSI -> unconnected-(A1-TX-Pad20)
- A1 pad 8: +5V -> unconnected-(A1-V+-Pad8)
- A1 pad 9: unconnected-(A1-VBat-Pad9) -> +5V
- U3 pad 5: HPM_RESET -> unconnected-(U3-RES-Pad5)
- U3 pad 6: UART_MISO -> TX
- U3 pad 7: UART_MOSI -> RX
Routing:
- net SDA: track 0.00 -> 93.7 mm
- net SCL: track 0.00 -> 75.1 mm
- net GND: track 0.00 -> 73.1 mm
- net UART_MOSI: track 69.4 -> 0.00 mm
- net UART_MISO: track 66.8 -> 0.00 mm
- net HPM_RESET: track 59.9 -> 0.00 mm
- net TX: track 0.00 -> 26.6 mm
- net RX: track 0.00 -> 24.2 mm
- net +3V3: track 8.18 -> 21.2 mm
- net +5V: track 122.4 -> 118.3 mm, vias 1 -> 0
- net unconnected-(A1-15-Pad14): track 0.00 -> 1.91 mm
Other:
- board text added: "MAKAYLA HOLDER INSTRUMENT SHOP"
- board text added: "REVISION C JULY 2023"
- board text removed: "BLAISE THOMPSON INSTRUMENT SHOP"
- board text removed: "REVISION B APRIL 2023"
