File: kicad/mqtt_particle_sensor.kicad_sch (KiCad schematic)
At the start: 21 parts, among them J2 Barrel_Jack, Q1 2N7000, Q2 2N7000, U1 CD4060BM96, U3 HPM_Particle_Sensor

Commit message: revC
Parts:
- added R8, R9: 4k7, Resistor_SMD:R_1206_3216Metric_Pad1.30x1.75mm_HandSolder, symbol Device:R_US
- added U2: ATtiny85-20P, Package_DIP:DIP-8_W7.62mm, symbol MCU_Microchip_ATtiny:ATtiny85-20P
Connections:
- net +3V3: now also R8.1, R9.1, U2.8 (VCC)
- net +5V: now also A1.9 (VBat); no longer A1.8 (V+)
- net GND: now also U2.4 (GND)
- net SDA: now reaches A1.17 (4)
- net SDA: now also R8.2, U2.5 (AREF/PB0)
- net SCL: now reaches A1.18 (5)
- net SCL: now also R9.2, U2.7 (PB2)
- net HPM_RESET: no longer names the net of U3.5 (RES)
- net HPM_RESET: no longer A1.14 (15)
- net UART_MISO: no longer names the net of A1.19 (RX)
- net UART_MISO: no longer U3.6 (TX)
- net UART_MOSI: no longer names the net of A1.20 (TX)
- net UART_MOSI: no longer U3.7 (RX)
- new net RX: U2.3 (XTAL2/PB4), U3.7 (RX)
- new net TX: U2.2 (XTAL1/PB3), U3.6 (TX)
- no-connect marks 21 -> 25
Other:
- note added: "ATtiny85"
